Commit message: ADD CPC sensor to the robot description
Signed-off-by: Musa Morena Marcusso Manhaes <Musa.Marcusso@de.bosch.com>

File: eca_a9_description/urdf/eca_a9_sensors.xacro (robot description, xacro)
@@ -105,3 +105,7 @@
       power_load="5"
       topic=""/>
+    <!-- Mount the chemical concentration sensor -->
+    <xacro:default_chemical_concentration_sensor namespace="${namespace}" parent_link="${namespace}/base_link">
+      <origin xyz="0 0 0" rpy="0 0 0"/>
+    </xacro:default_chemical_concentration_sensor>
 </robot>
