Commit message: ADD Sliding mode control files (still experimental)
Signed-off-by: Musa Morena Marcusso Manhaes <Musa.Marcusso@de.bosch.com>

File: eca_a9_description/urdf/eca_a9_snippets.xacro (robot description, xacro)
@@ -13,14 +13,39 @@
 -->
 <robot xmlns:xacro="http://www.ros.org/wiki/xacro">
+    <xacro:property name="fin_area" value="0.04155"/>
+    <xacro:property name="fin_drag_coef" value="0.04155"/>
+    <xacro:property name="fin_lift_coef" value="3.0"/>
+    <xacro:property name="fin_rho" value="1028.0"/>
     <!-- FIN SNIPPETS -->
     <xacro:macro name="fin_macro" params="namespace fin_id *origin">
+      <xacro:fin_two_lines_macro
+        namespace="${namespace}"
+        parent_link="${namespace}/base_link"
+        fin_id="${fin_id}"
+        min_joint_limit="${-80*d2r}"
+        max_joint_limit="${80*d2r}"
+        mesh_filename="${fin_mesh_file}"
+        fin_dynamics_time_constant="0.1"
+        fin_cross_section_area="0.04155"
+        current_velocity_topic="current_velocity"
+        fluid_density="1027.0"
+        a0="0.0"
+        alpha_stall="0.174533"
+        cla="13.98"
+        cla_stall="0.0"
+        cda="0.0"
+        cda_stall="">
+        <xacro:insert_block name="origin"/>
+      </xacro:fin_two_lines_macro>
+    </xacro:macro>
+    <!-- <xacro:macro name="fin_macro" params="namespace fin_id *origin">
       <xacro:fin_quadratic_macro
         namespace="${namespace}"
         parent_link="${namespace}/base_link"
         fin_id="${fin_id}"
-        min_joint_limit="${-90*d2r}"
-        max_joint_limit="${90*d2r}"
+        min_joint_limit="${-45*d2r}"
+        max_joint_limit="${45*d2r}"
         mesh_filename="${fin_mesh_file}"
-        fin_dynamics_time_constant="0.2"
+        fin_dynamics_time_constant="0.1"
         lift_constant="7.2"
         drag_constant="6.3"
@@ -28,4 +53,4 @@
         <xacro:insert_block name="origin"/>
       </xacro:fin_quadratic_macro>
-    </xacro:macro>
+    </xacro:macro> -->
 </robot>
