Commit message: FIX Instance of Pose 3D sensor with inertial frame reference
Signed-off-by: Musa Morena Marcusso Manhaes <Musa.Marcusso@de.bosch.com>

File: eca_a9_description/robots/eca_a9_default.urdf.xacro (robot description, xacro)
@@ -15,8 +15,12 @@
   <xacro:arg name="debug" default="0"/>
   <xacro:arg name="namespace" default="eca_a9"/>
+  <xacro:arg name="inertial_reference_frame" default="world"/>
   <!-- Include the UUV macro file -->
   <xacro:include filename="$(find eca_a9_description)/urdf/eca_a9_base.xacro"/>
   <!-- Create the eca_a9 -->
-  <xacro:eca_a9_base namespace="$(arg namespace)" debug="$(arg debug)"/>
+  <xacro:eca_a9_base
+    namespace="$(arg namespace)"
+    debug="$(arg debug)"
+    inertial_reference_frame="$(arg inertial_reference_frame)"/>
   <!-- Joint state publisher plugin -->
   <gazebo>

File: eca_a9_description/urdf/eca_a9_base.xacro (robot description, xacro)
@@ -32,5 +32,5 @@
   <xacro:property name="prop_mesh_file" value="file://$(find eca_a9_description)/mesh/eca_a9_propeller.dae"/>
   <xacro:property name="fin_mesh_file" value="file://$(find eca_a9_description)/mesh/eca_a9_fin.dae"/>
-  <xacro:macro name="eca_a9_base" params="namespace debug">
+  <xacro:macro name="eca_a9_base" params="namespace debug inertial_reference_frame">
     <link name="${namespace}/base_link">
       <visual>

File: eca_a9_description/urdf/eca_a9_sensors.xacro (robot description, xacro)
@@ -14,5 +14,8 @@
 <robot xmlns:xacro="http://www.ros.org/wiki/xacro">
     <!-- Mount a 3D pose sensor -->
-    <xacro:default_pose_3d namespace="${namespace}" parent_link="${namespace}/base_link" />
+    <xacro:default_pose_3d_macro
+      namespace="${namespace}"
+      parent_link="${namespace}/base_link"
+      inertial_reference_frame="${inertial_reference_frame}" />
     <!-- DVL sensor -->
     <xacro:dvl_plugin_macro
